Commit message: restart

File: catkin_ws/src/my_robot/urdf/my_robot.xacro (robot description, xacro)
@@ -183,5 +183,5 @@
 <joint name="camera_optical_joint" type="fixed">
   <origin xyz="0 0 0" rpy="-1.5707 0 -1.5707"/>
-  <parent link="camera_link"/>
+  <parent link="camera"/>
   <child link="camera_link_optical"/>
 </joint>
